File: Hardware/SunriseLamp.kicad_pcb (KiCad board)
At the start: 2 copper layers, 0 parts

Commit message: Most part assignents made, pending switch footprint & xtal selection
Parts:
- added C1: 2u2 100V, Capacitor_SMD:CP_Elec_6.3x5.4, F.Cu at (133.0, 104.0)
- added C10: 2u2 100V, Capacitor_SMD:CP_Elec_6.3x5.4, F.Cu at (152.6, 82.4)
- added C11: 4u7 100V, Capacitor_SMD:C_1210_3225Metric, F.Cu at (187.6, 65.4)
- added C12: 10u 25V, Capacitor_SMD:C_0805_2012Metric_Pad1.18x1.45mm_HandSolder, F.Cu at (120.2, 113.0)
- added C13: 47u 25V, Capacitor_SMD:CP_Elec_6.3x5.4, F.Cu at (155.1, 72.4)
- added C14: 1u 16V, Capacitor_SMD:C_0805_2012Metric_Pad1.18x1.45mm_HandSolder, F.Cu at (110.6, 113.0)
- added C15: 2u2 100V, Capacitor_SMD:CP_Elec_6.3x5.4, F.Cu at (165.7, 72.4)
- added C16: 1u 16V, Capacitor_SMD:C_0805_2012Metric_Pad1.18x1.45mm_HandSolder, F.Cu at (101.0, 113.0)
- added C17: 22u TANT, Capacitor_Tantalum_SMD:CP_EIA-3528-15_AVX-H, F.Cu at (160.4, 92.8)
- added C18: 22p, Capacitor_SMD:C_0805_2012Metric_Pad1.18x1.45mm_HandSolder, F.Cu at (130.6, 126.8)
- added C19: 22p, Capacitor_SMD:C_0805_2012Metric_Pad1.18x1.45mm_HandSolder, F.Cu at (135.5, 119.4)
- added C2: 1u 16V, Capacitor_SMD:C_0805_2012Metric_Pad1.18x1.45mm_HandSolder, F.Cu at (115.4, 113.0)
- added C20: 100n, Capacitor_SMD:C_0805_2012Metric_Pad1.18x1.45mm_HandSolder, F.Cu at (135.5, 122.4)
- added C21: 1u, Capacitor_SMD:C_0805_2012Metric_Pad1.18x1.45mm_HandSolder, F.Cu at (117.0, 142.8)
- added C22: 100n, Capacitor_SMD:C_0805_2012Metric_Pad1.18x1.45mm_HandSolder, F.Cu at (130.6, 123.8)
- added C23: 22u, Capacitor_SMD:C_0805_2012Metric_Pad1.18x1.45mm_HandSolder, F.Cu at (124.5, 134.7)
- added C24: 100n, Capacitor_SMD:C_0805_2012Metric_Pad1.18x1.45mm_HandSolder, F.Cu at (124.5, 131.7)
- added C25: 100n, Capacitor_SMD:C_0805_2012Metric_Pad1.18x1.45mm_HandSolder, F.Cu at (117.0, 139.8)
- added C26: 10u 25V, Capacitor_SMD:C_0805_2012Metric_Pad1.18x1.45mm_HandSolder, F.Cu at (124.5, 128.6)
- added C27: 100n, Capacitor_SMD:C_0805_2012Metric_Pad1.18x1.45mm_HandSolder, F.Cu at (118.1, 135.4)
- added C28: 1u, Capacitor_SMD:C_0805_2012Metric_Pad1.18x1.45mm_HandSolder, F.Cu at (140.3, 119.4)
- added C3: 10nF 50V, Capacitor_SMD:C_0805_2012Metric_Pad1.18x1.45mm_HandSolder, F.Cu at (149.6, 88.0)
- added C4: 4u7 100V, Capacitor_SMD:C_1210_3225Metric, F.Cu at (151.2, 103.0)
- added C5: 10u 25V, Capacitor_SMD:C_0805_2012Metric_Pad1.18x1.45mm_HandSolder, F.Cu at (166.7, 66.4)
- added C6: 47u 25V, Capacitor_SMD:CP_Elec_6.3x5.4, F.Cu at (138.0, 94.0)
- added C7: 2u2 100V, Capacitor_SMD:CP_Elec_6.3x5.4, F.Cu at (169.6, 60.9)
- added C8: 1u 16V, Capacitor_SMD:C_0805_2012Metric_Pad1.18x1.45mm_HandSolder, F.Cu at (145.7, 96.0)
- added C9: 10nF 50V, Capacitor_SMD:C_0805_2012Metric_Pad1.18x1.45mm_HandSolder, F.Cu at (105.8, 113.0)
- added D1: SS310, Diode_SMD:D_SMA_Handsoldering, F.Cu at (132.7, 110.3)
- added D2: SS310, Diode_SMD:D_SMA_Handsoldering, F.Cu at (148.3, 92.2)
- added D3: SS310, Diode_SMD:D_SMA_Handsoldering, F.Cu at (143.3, 100.3)
- added D4: SS310, Diode_SMD:D_SMA_Handsoldering, F.Cu at (162.9, 78.8)
- added D5: SS34, Diode_SMD:D_SMA_Handsoldering, F.Cu at (179.9, 59.1)
- added D6: SS34, Diode_SMD:D_SMA_Handsoldering, F.Cu at (103.6, 141.6)
- added D7: GREEN, LED_SMD:LED_0603_1608Metric_Pad1.05x0.95mm_HandSolder, F.Cu at (121.6, 138.2)
- added D8: RED, LED_SMD:LED_0603_1608Metric_Pad1.05x0.95mm_HandSolder, F.Cu at (110.8, 143.9)
- added F1: 0ZCJ0050FF2G, Fuse:Fuse_1206_3216Metric_Pad1.42x1.75mm_HandSolder, F.Cu at (111.6, 140.9)
- added J1: Molex 047053-1000, Connector_Molex:Molex_KK-254_AE-6410-04A_1x04_P2.54mm_Vertical, F.Cu at (100.9, 135.4)
- added J2: S3B-XH-A, Connector_JST:JST_XH_S3B-XH-A-1_1x03_P2.50mm_Horizontal, F.Cu at (102.0, 122.8)
- added L1: 33u 2A, Inductor_SMD:L_SigTra_SC3316F, F.Cu at (120.4, 105.7)
- added L2: 20uH >1.2A, Inductor_SMD:L_Taiyo-Yuden_NR-80xx, F.Cu at (143.1, 107.4)
- added L3: 33u 2A, Inductor_SMD:L_SigTra_SC3316F, F.Cu at (105.8, 105.7)
- added L4: 20uH >0.5A, Inductor_SMD:L_Taiyo-Yuden_NR-80xx, F.Cu at (162.7, 85.8)
- added L5: 33u 2A, Inductor_SMD:L_SigTra_SC3316F, F.Cu at (157.0, 62.6)
- added L6: 33u 2A, Inductor_SMD:L_SigTra_SC3316F, F.Cu at (139.9, 84.1)
- added P1: XT60PW-M, PersonalConnectors:AMASS_XT60PW-M, F.Cu at (124.2, 89.5)
- added P2: XT60PW-F, PersonalConnectors:AMASS_XT60PW-F, F.Cu at (107.1, 89.5)
- added P3: XT60PW-F, PersonalConnectors:AMASS_XT60PW-F, F.Cu at (124.2, 67.9)
- added P4: XT60PW-F, PersonalConnectors:AMASS_XT60PW-F, F.Cu at (141.2, 67.9)
- added P5: XT60PW-F, PersonalConnectors:AMASS_XT60PW-F, F.Cu at (107.1, 67.9)
- added Q1: MMBT3904, Package_TO_SOT_SMD:SOT-23, F.Cu at (130.7, 120.1)
- added Q2: MMBT3904, Package_TO_SOT_SMD:SOT-23, F.Cu at (119.7, 131.6)
- added Q3: PMV16XNR, Package_TO_SOT_SMD:SOT-23_Handsoldering, F.Cu at (114.0, 131.6)
- added Q4: MMBT3904, Package_TO_SOT_SMD:SOT-23, F.Cu at (113.2, 136.1)
- added R1: 3k3, Resistor_SMD:R_0603_1608Metric_Pad0.98x0.95mm_HandSolder, F.Cu at (187.4, 68.7)
- added R10: 100k, Resistor_SMD:R_0603_1608Metric_Pad0.98x0.95mm_HandSolder, F.Cu at (179.2, 77.3)
- added R11: 33k, Resistor_SMD:R_0603_1608Metric_Pad0.98x0.95mm_HandSolder, F.Cu at (173.9, 84.2)
- added R12: 22k, Resistor_SMD:R_0603_1608Metric_Pad0.98x0.95mm_HandSolder, F.Cu at (171.3, 66.2)
- added R13: 3k3, Resistor_SMD:R_0603_1608Metric_Pad0.98x0.95mm_HandSolder, F.Cu at (169.6, 84.2)
- added R14: 20k, Resistor_SMD:R_0603_1608Metric_Pad0.98x0.95mm_HandSolder, F.Cu at (139.9, 113.4)
- added R15: 3k3, Resistor_SMD:R_0603_1608Metric_Pad0.98x0.95mm_HandSolder, F.Cu at (165.6, 91.8)
- added R16: 20k, Resistor_SMD:R_0603_1608Metric_Pad0.98x0.95mm_HandSolder, F.Cu at (156.2, 102.2)
- added R17: 5k1, Resistor_SMD:R_0603_1608Metric_Pad0.98x0.95mm_HandSolder, F.Cu at (135.2, 125.2)
- added R18: 5k1, Resistor_SMD:R_0603_1608Metric_Pad0.98x0.95mm_HandSolder, F.Cu at (139.6, 125.2)
- added R19: 4k7, Resistor_SMD:R_0603_1608Metric_Pad0.98x0.95mm_HandSolder, F.Cu at (140.1, 122.2)
- added R2: 20k, Resistor_SMD:R_0603_1608Metric_Pad0.98x0.95mm_HandSolder, F.Cu at (144.2, 113.4)
- added R20: 3k3, Resistor_SMD:R_0603_1608Metric_Pad0.98x0.95mm_HandSolder, F.Cu at (129.1, 132.1)
- added R21: 10k, Resistor_SMD:R_0603_1608Metric_Pad0.98x0.95mm_HandSolder, F.Cu at (121.6, 140.7)
- added R22: 0R, Resistor_SMD:R_0603_1608Metric_Pad0.98x0.95mm_HandSolder, F.Cu at (129.1, 134.6)
- added R23: 0R, Resistor_SMD:R_0603_1608Metric_Pad0.98x0.95mm_HandSolder, F.Cu at (144.4, 122.2)
- added R24: 10k, Resistor_SMD:R_0603_1608Metric_Pad0.98x0.95mm_HandSolder, F.Cu at (121.6, 143.2)
- added R25: 10k, Resistor_SMD:R_0603_1608Metric_Pad0.98x0.95mm_HandSolder, F.Cu at (126.0, 139.9)
- added R26: 2k7, Resistor_SMD:R_0603_1608Metric_Pad0.98x0.95mm_HandSolder, F.Cu at (125.9, 142.4)
- added R27: 1k, Resistor_SMD:R_0603_1608Metric_Pad0.98x0.95mm_HandSolder, F.Cu at (144.9, 119.1)
- added R28: 10k, Resistor_SMD:R_0603_1608Metric_Pad0.98x0.95mm_HandSolder, F.Cu at (126.0, 137.4)
- added R29: NF, Resistor_SMD:R_0603_1608Metric_Pad0.98x0.95mm_HandSolder, F.Cu at (133.5, 129.6)
- added R3: 100k, Resistor_SMD:R_0603_1608Metric_Pad0.98x0.95mm_HandSolder, F.Cu at (169.6, 86.7)
- added R30: 4k7, Resistor_SMD:R_0603_1608Metric_Pad0.98x0.95mm_HandSolder, F.Cu at (129.1, 129.6)
- added R31: 4k7, Resistor_SMD:R_0603_1608Metric_Pad0.98x0.95mm_HandSolder, F.Cu at (133.5, 132.1)
- added R4: 4k7, Resistor_SMD:R_0603_1608Metric_Pad0.98x0.95mm_HandSolder, F.Cu at (159.6, 98.7)
- added R5: 100k, Resistor_SMD:R_0603_1608Metric_Pad0.98x0.95mm_HandSolder, F.Cu at (124.8, 112.7)
- added R6: 560R, Resistor_SMD:R_0603_1608Metric_Pad0.98x0.95mm_HandSolder, F.Cu at (192.6, 64.5)
- added R7: 3k3, Resistor_SMD:R_0603_1608Metric_Pad0.98x0.95mm_HandSolder, F.Cu at (150.1, 106.4)
- added R8: 20k, Resistor_SMD:R_0603_1608Metric_Pad0.98x0.95mm_HandSolder, F.Cu at (159.6, 96.2)
- added R9: 100k, Resistor_SMD:R_0603_1608Metric_Pad0.98x0.95mm_HandSolder, F.Cu at (154.2, 87.8)
- added U1: LM3414, PersonalDiscretes:TI_SO-PowerPAD-8_HandSolder, F.Cu at (152.9, 97.7)
- added U2: SY8303, Package_TO_SOT_SMD:TSOT-23-8, F.Cu at (196.6, 59.0)
- added U3: LM3414, PersonalDiscretes:TI_SO-PowerPAD-8_HandSolder, F.Cu at (189.5, 60.0)
- added U4: SY8303, Package_TO_SOT_SMD:TSOT-23-8, F.Cu at (182.7, 71.8)
- added U5: LM3414, PersonalDiscretes:TI_SO-PowerPAD-8_HandSolder, F.Cu at (172.4, 79.7)
- added U6: AMS1117-3.3, Package_TO_SOT_SMD:SOT-223-3_TabPin2, F.Cu at (179.8, 65.5)
- added U7: LM3414, PersonalDiscretes:TI_SO-PowerPAD-8_HandSolder, F.Cu at (175.6, 72.8)
- added U8: CH340G, Package_SO:SOIC-16_3.9x9.9mm_P1.27mm, F.Cu at (114.8, 123.6)
- added U9: ESP32-PICO-MINI-02, Package_DFN_QFN:QFN-48-1EP_7x7mm_P0.5mm_EP5.3x5.3mm, F.Cu at (123.6, 122.5)
