File: Hardware/SunriseLamp.kicad_pcb (KiCad board)
At the start: 2 copper layers, 94 parts, among them J1 Molex 047053-1000, J2 S3B-XH-A, P1 XT60PW-M, P2 XT60PW-F, P3 XT60PW-F, P4 XT60PW-F, P5 XT60PW-F, Q1 MMBT3904, Q2 MMBT3904, Q3 PMV16XNR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

Commit message: USB footprint added, mount holes added.
Parts:
- added H1: 3.2mm, MountingHole:MountingHole_3.2mm_M3_DIN965_Pad, F.Cu at (79.0, 123.0)
- added H2: 3.2mm, MountingHole:MountingHole_3.2mm_M3_DIN965_Pad, F.Cu at (86.2, 123.0)
- added H3: 3.2mm, MountingHole:MountingHole_3.2mm_M3_DIN965_Pad, F.Cu at (86.2, 130.2)
- added H4: 3.2mm, MountingHole:MountingHole_3.2mm_M3_DIN965_Pad, F.Cu at (79.0, 130.2)
- added P6: TYPE-C-31-M-12, PersonalConnectors:Korean_HRO_Type-C-31-M-12, F.Cu at (116.5, 68.9)
- added R32: 0R, Resistor_SMD:R_0805_2012Metric_Pad1.20x1.40mm_HandSolder, F.Cu at (96.8, 120.9)
- added R33: 0R, Resistor_SMD:R_0805_2012Metric_Pad1.20x1.40mm_HandSolder, F.Cu at (92.1, 123.8)
- added R34: 0R, Resistor_SMD:R_0805_2012Metric_Pad1.20x1.40mm_HandSolder, F.Cu at (92.1, 120.9)
- added R35: 0R, Resistor_SMD:R_0805_2012Metric_Pad1.20x1.40mm_HandSolder, F.Cu at (92.1, 126.8)
- added Y1: 12MHz, Crystal:Crystal_SMD_3225-4Pin_3.2x2.5mm, F.Cu at (128.7, 64.4)
- moved P5 134.4 mm to (231.0, 120.0), turned to -90 degrees
- moved P2 132.3 mm to (231.0, 136.0), turned to -90 degrees
- moved P3 112.8 mm to (231.0, 104.0), turned to -90 degrees
- moved P4 92.0 mm to (231.0, 88.0), turned to -90 degrees
- moved Q3 69.1 mm to (54.5, 96.5)
- moved R29 69.1 mm to (74.0, 94.5)
- moved R30 69.1 mm to (69.7, 94.5)
- moved C1 69.1 mm to (73.5, 68.9)
- moved C10 69.1 mm to (93.1, 47.3)
- moved C11 69.1 mm to (128.1, 30.2)
- moved C13 69.1 mm to (95.6, 37.3)
- moved C14 69.1 mm to (51.1, 77.9)
- moved C17 69.1 mm to (101.0, 57.6)
- moved C19 69.1 mm to (76.1, 84.3)
- moved C2 69.1 mm to (56.0, 77.9)
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Other:
- board outline added: 80 x 80 mm

Commit message: Whoops, acidentally wiped all part assignments somehow. corrected.
Only pending footprint creation is for two switches.
Parts:
- H1, H2, H3, H4: value 3.2mm -> 4.3mm; footprint MountingHole:MountingHole_3.2mm_M3_DIN965_Pad -> MountingHole:MountingHole_4.3mm_M4_DIN965_Pad_TopBottom
Changed lines of the file:
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@@
     )
   )
-  (footprint "MountingHole:MountingHole_3.2mm_M3_DIN965_Pad" (layer "F.Cu")
+  (footprint "MountingHole:MountingHole_4.3mm_M4_DIN965_Pad_TopBottom" (layer "F.Cu")
     (at 79 123)
-    (descr "Mounting Hole 3.2mm, M3, DIN965")
-    (tags "mounting hole 3.2mm m3 din965")
+    (descr "Mounting Hole 4.3mm, M4, DIN965")
+    (tags "mounting hole 4.3mm m4 din965")
     (property "Sheetfile" "SunriseLamp.kicad_sch")
     (property "Sheetname" "")
     (attr exclude_from_pos_files)
-    (fp_text reference "H1" (at 0 -3.8) (layer "F.SilkS")
-      (effects (font (size 1 1) (thickness 0.15)))
-    )
-    (fp_text value "3.2mm" (at 0 3.8) (layer "F.Fab")
-      (effects (font (size 1 1) (thickness 0.15)))
-    )
-    (fp_text user "${REFERENCE}" (at 0 0) (layer "F.Fab")
-      (effects (font (size 1 1) (thickness 0.15)))
-    )
-    (fp_circle (center 0 0) (end 2.8 0) (layer "Cmts.User") (width 0.15) (fill none))
-    (fp_circle (center 0 0) (end 3.05 0) (layer "F.CrtYd") (width 0.05) (fill none))
-    (pad "1" thru_hole circle (at 0 0) (size 5.6 5.6) (drill 3.2) (layers *.Cu *.Mask)
+    (fp_text reference "H1" (at 0 -4.75) (layer "F.SilkS")
+      (effects (font (size 1 1) (thickness 0.15)))
+    )
+    (fp_text value "4.3mm" (at 0 4.75) (layer "F.Fab")
+      (effects (font (size 1 1) (thickness 0.15)))
+    )
+    (fp_text user "${REFERENCE}" (at 0 0) (layer "F.Fab")
+      (effects (font (size 1 1) (thickness 0.15)))
+    )
+    (fp_circle (center 0 0) (end 3.75 0) (layer "Cmts.User") (width 0.15) (fill none))
+    (fp_circle (center 0 0) (end 4 0) (layer "F.CrtYd") (width 0.05) (fill none))
+    (pad "1" connect circle (at 0 0) (size 7.5 7.5) (layers "F.Cu" "F.Mask")
+      (net 98 "Net-(H1-Pad1)") (pinfunction "1") (pintype "input"))
+    (pad "1" connect circle (at 0 0) (size 7.5 7.5) (layers "B.Cu" "B.Mask")
+      (net 98 "Net-(H1-Pad1)") (pinfunction "1") (pintype "input"))
+    (pad "1" thru_hole circle (at 0 0) (size 4.7 4.7) (drill 4.3) (layers *.Cu *.Mask)
       (net 98 "Net-(H1-Pad1)") (pinfunction "1") (pintype "input"))
   )
@@
     )
   )
-  (footprint "MountingHole:MountingHole_3.2mm_M3_DIN965_Pad" (layer "F.Cu")
+  (footprint "MountingHole:MountingHole_4.3mm_M4_DIN965_Pad_TopBottom" (layer "F.Cu")
     (at 86.15 130.15)
-    (descr "Mounting Hole 3.2mm, M3, DIN965")
-    (tags "mounting hole 3.2mm m3 din965")
+    (descr "Mounting Hole 4.3mm, M4, DIN965")
+    (tags "mounting hole 4.3mm m4 din965")
     (property "Sheetfile" "SunriseLamp.kicad_sch")
     (property "Sheetname" "")
     (attr exclude_from_pos_files)
-    (fp_text reference "H3" (at 0 -3.8) (layer "F.SilkS")
-      (effects (font (size 1 1) (thickness 0.15)))
-    )
-    (fp_text value "3.2mm" (at 0 3.8) (layer "F.Fab")
-      (effects (font (size 1 1) (thickness 0.15)))
-    )
-    (fp_text user "${REFERENCE}" (at 0 0) (layer "F.Fab")
-      (effects (font (size 1 1) (thickness 0.15)))
-    )
-    (fp_circle (center 0 0) (end 2.8 0) (layer "Cmts.User") (width 0.15) (fill none))
-    (fp_circle (center 0 0) (end 3.05 0) (layer "F.CrtYd") (width 0.05) (fill none))
-    (pad "1" thru_hole circle (at 0 0) (size 5.6 5.6) (drill 3.2) (layers *.Cu *.Mask)
+    (fp_text reference "H3" (at 0 -4.75) (layer "F.SilkS")
+      (effects (font (size 1 1) (thickness 0.15)))
+    )
+    (fp_text value "4.3mm" (at 0 4.75) (layer "F.Fab")
+      (effects (font (size 1 1) (thickness 0.15)))
+    )
+    (fp_text user "${REFERENCE}" (at 0 0) (layer "F.Fab")
+      (effects (font (size 1 1) (thickness 0.15)))
+    )
+    (fp_circle (center 0 0) (end 3.75 0) (layer "Cmts.User") (width 0.15) (fill none))
+    (fp_circle (center 0 0) (end 4 0) (layer "F.CrtYd") (width 0.05) (fill none))
+    (pad "1" thru_hole circle (at 0 0) (size 4.7 4.7) (drill 4.3) (layers *.Cu *.Mask)
+      (net 100 "Net-(H3-Pad1)") (pinfunction "1") (pintype "input"))
+    (pad "1" connect circle (at 0 0) (size 7.5 7.5) (layers "B.Cu" "B.Mask")
+      (net 100 "Net-(H3-Pad1)") (pinfunction "1") (pintype "input"))
+    (pad "1" connect circle (at 0 0) (size 7.5 7.5) (layers "F.Cu" "F.Mask")
       (net 100 "Net-(H3-Pad1)") (pinfunction "1") (pintype "input"))
   )
@@
     )
   )
-  (footprint "MountingHole:MountingHole_3.2mm_M3_DIN965_Pad" (layer "F.Cu")
+  (footprint "MountingHole:MountingHole_4.3mm_M4_DIN965_Pad_TopBottom" (layer "F.Cu")
     (at 86.15 123)
-    (descr "Mounting Hole 3.2mm, M3, DIN965")
-    (tags "mounting hole 3.2mm m3 din965")
+    (descr "Mounting Hole 4.3mm, M4, DIN965")
+    (tags "mounting hole 4.3mm m4 din965")
     (property "Sheetfile" "SunriseLamp.kicad_sch")
     (property "Sheetname" "")
     (attr exclude_from_pos_files)
-    (fp_text reference "H2" (at 0 -3.8) (layer "F.SilkS")
-      (effects (font (size 1 1) (thickness 0.15)))
-    )
-    (fp_text value "3.2mm" (at 0 3.8) (layer "F.Fab")
-      (effects (font (size 1 1) (thickness 0.15)))
-    )
-    (fp_text user "${REFERENCE}" (at 0 0) (layer "F.Fab")
-      (effects (font (size 1 1) (thickness 0.15)))
-    )
-    (fp_circle (center 0 0) (end 2.8 0) (layer "Cmts.User") (width 0.15) (fill none))
-    (fp_circle (center 0 0) (end 3.05 0) (layer "F.CrtYd") (width 0.05) (fill none))
-    (pad "1" thru_hole circle (at 0 0) (size 5.6 5.6) (drill 3.2) (layers *.Cu *.Mask)
+    (fp_text reference "H2" (at 0 -4.75) (layer "F.SilkS")
+      (effects (font (size 1 1) (thickness 0.15)))
+    )
+    (fp_text value "4.3mm" (at 0 4.75) (layer "F.Fab")
+      (effects (font (size 1 1) (thickness 0.15)))
+    )
+    (fp_text user "${REFERENCE}" (at 0 0) (layer "F.Fab")
+      (effects (font (size 1 1) (thickness 0.15)))
+    )
+    (fp_circle (center 0 0) (end 3.75 0) (layer "Cmts.User") (width 0.15) (fill none))
+    (fp_circle (center 0 0) (end 4 0) (layer "F.CrtYd") (width 0.05) (fill none))
+    (pad "1" connect circle (at 0 0) (size 7.5 7.5) (layers "B.Cu" "B.Mask")
+      (net 99 "Net-(H2-Pad1)") (pinfunction "1") (pintype "input"))
+    (pad "1" thru_hole circle (at 0 0) (size 4.7 4.7) (drill 4.3) (layers *.Cu *.Mask)
+      (net 99 "Net-(H2-Pad1)") (pinfunction "1") (pintype "input"))
+    (pad "1" connect circle (at 0 0) (size 7.5 7.5) (layers "F.Cu" "F.Mask")
       (net 99 "Net-(H2-Pad1)") (pinfunction "1") (pintype "input"))
   )
@@
     )
   )
-  (footprint "MountingHole:MountingHole_3.2mm_M3_DIN965_Pad" (layer "F.Cu")
+  (footprint "MountingHole:MountingHole_4.3mm_M4_DIN965_Pad_TopBottom" (layer "F.Cu")
     (at 79 130.15)
-    (descr "Mounting Hole 3.2mm, M3, DIN965")
-    (tags "mounting hole 3.2mm m3 din965")
+    (descr "Mounting Hole 4.3mm, M4, DIN965")
+    (tags "mounting hole 4.3mm m4 din965")
     (property "Sheetfile" "SunriseLamp.kicad_sch")
     (property "Sheetname" "")
     (attr exclude_from_pos_files)
-    (fp_text reference "H4" (at 0 -3.8) (layer "F.SilkS")
-      (effects (font (size 1 1) (thickness 0.15)))
-    )
-    (fp_text value "3.2mm" (at 0 3.8) (layer "F.Fab")
-      (effects (font (size 1 1) (thickness 0.15)))
-    )
-    (fp_text user "${REFERENCE}" (at 0 0) (layer "F.Fab")
-      (effects (font (size 1 1) (thickness 0.15)))
-    )
-    (fp_circle (center 0 0) (end 2.8 0) (layer "Cmts.User") (width 0.15) (fill none))
-    (fp_circle (center 0 0) (end 3.05 0) (layer "F.CrtYd") (width 0.05) (fill none))
-    (pad "1" thru_hole circle (at 0 0) (size 5.6 5.6) (drill 3.2) (layers *.Cu *.Mask)
+    (fp_text reference "H4" (at 0 -4.75) (layer "F.SilkS")
+      (effects (font (size 1 1) (thickness 0.15)))
+    )
+    (fp_text value "4.3mm" (at 0 4.75) (layer "F.Fab")
+      (effects (font (size 1 1) (thickness 0.15)))
+    )
+    (fp_text user "${REFERENCE}" (at 0 0) (layer "F.Fab")
+      (effects (font (size 1 1) (thickness 0.15)))
+    )
+    (fp_circle (center 0 0) (end 3.75 0) (layer "Cmts.User") (width 0.15) (fill none))
+    (fp_circle (center 0 0) (end 4 0) (layer "F.CrtYd") (width 0.05) (fill none))
+    (pad "1" connect circle (at 0 0) (size 7.5 7.5) (layers "B.Cu" "B.Mask")
       (net 101 "Net-(H4-Pad1)") (pinfunction "1") (pintype "input"))
-  )
+    (pad "1" connect circle (at 0 0) (size 7.5 7.5) (layers "F.Cu" "F.Mask")
+      (net 101 "Net-(H4-Pad1)") (pinfunction "1") (pintype "input"))
+    (pad "1" thru_hole circle (at 0 0) (size 4.7 4.7) (drill 4.3) (layers *.Cu *.Mask)
+      (net 101 "Net-(H4-Pad1)") (pinfunction "1") (pintype "input"))
+  )

Commit message: Layout changes
Changed XT60 outputs to Mini-Fit Jr., laid out 80mm fan edge cuts, started positioning conns
Parts:
- removed P2, P3, P4, P5: XT60PW-F, PersonalConnectors:AMASS_XT60PW-F
- added J3: Molex 26013114, Connector_Molex:Molex_Mini-Fit_Jr_5569-02A2_2x01_P4.20mm_Horizontal, F.Cu at (216.2, 87.5)
- added J4: Molex 26013114, Connector_Molex:Molex_Mini-Fit_Jr_5569-02A2_2x01_P4.20mm_Horizontal, F.Cu at (216.2, 104.0)
- added J5: Molex 26013114, Connector_Molex:Molex_Mini-Fit_Jr_5569-02A2_2x01_P4.20mm_Horizontal, F.Cu at (216.2, 120.5)
- added J6: Molex 26013114, Connector_Molex:Molex_Mini-Fit_Jr_5569-02A2_2x01_P4.20mm_Horizontal, F.Cu at (216.2, 137.0)
- moved H2 147.9 mm to (225.8, 74.2)
- moved J2 142.4 mm to (174.0, 142.6)
- moved H3 140.5 mm to (225.8, 145.8)
- moved U8 116.5 mm to (162.0, 135.2), turned to 90 degrees
- moved P1 101.9 mm to (160.5, 89.0), turned to 90 degrees
- moved U9 99.9 mm to (124.8, 166.8)
- moved P6 92.8 mm to (165.2, 147.9)
- moved H1 89.7 mm to (154.2, 74.2)
- moved H4 76.8 mm to (154.2, 145.8)
Other:
- outline, holes or cut-outs redrawn
- copper layers 2 -> 4

Commit message: removing white channel -- limited space on side of board from inductors
Parts:
- removed C15: 2u2 100V, Capacitor_SMD:CP_Elec_6.3x5.4
- removed C16: 1u 16V, Capacitor_SMD:C_0805_2012Metric_Pad1.18x1.45mm_HandSolder
- removed D4: SS310, Diode_SMD:D_SMA_Handsoldering
- removed J6: Molex 26013114, Connector_Molex:Molex_Mini-Fit_Jr_5569-02A2_2x01_P4.20mm_Horizontal
- removed L6: 33u 2A, Inductor_SMD:L_SigTra_SC3316F
- removed R15: 3k3, Resistor_SMD:R_0603_1608Metric_Pad0.98x0.95mm_HandSolder
- removed R16: 20k, Resistor_SMD:R_0603_1608Metric_Pad0.98x0.95mm_HandSolder
- removed U7: LM3414, PersonalDiscretes:TI_SO-PowerPAD-8_HandSolder
- L1, L3, L5: footprint Inductor_SMD:L_SigTra_SC3316F -> Inductor_SMD:L_12x12mm_H6mm
- moved C28 874.9 mm to (579.1, 803.4)
- moved C27 863.7 mm to (560.1, 803.4)
- moved J1 833.0 mm to (542.9, 765.3)
- moved Q3 832.8 mm to (529.6, 780.6)
- moved R28 820.8 mm to (514.4, 790.1)
- moved R27 811.1 mm to (501.0, 780.6)
- moved C22 766.9 mm to (287.7, 824.4)
- moved Q4 764.1 mm to (504.8, 717.7)
- moved C23 762.9 mm to (302.9, 824.4)
- moved R26 759.8 mm to (468.6, 752.0)
- moved R30 748.3 mm to (483.9, 717.7)
- moved R29 742.7 mm to (508.6, 696.8)
- moved Q2 740.6 mm to (102.9, 835.8)
- moved R25 731.1 mm to (74.3, 835.8)
- moved Q1 715.3 mm to (102.9, 799.6)
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Connections:
- J3 pad 1: +36V -> Net-(L1-Pad2)
- J3 pad 2: Net-(L1-Pad2) -> +36V
- J4 pad 1: +36V -> Net-(L3-Pad2)
- J4 pad 2: Net-(L3-Pad2) -> +36V
- J5 pad 1: +36V -> Net-(J5-Pad1)
- J5 pad 2: Net-(L5-Pad2) -> +36V
- L5 pad 2: Net-(L5-Pad2) -> Net-(J5-Pad1)

Commit message: adding back in 4th channel -- maybe still RGBW?
Parts:
- moved C10 352.5 mm to (197.8, 120.8)
- moved C7 326.3 mm to (197.7, 99.0)
- moved D3 306.0 mm to (204.5, 124.8), turned to -90 degrees
- moved R14 304.2 mm to (203.5, 130.2)
- moved U5 281.8 mm to (197.6, 127.8)
- moved D2 275.5 mm to (204.5, 103.0), turned to -90 degrees
- moved R13 275.4 mm to (191.5, 128.5), turned to 180 degrees
- moved R8 267.4 mm to (203.5, 108.5)
- moved C14 260.5 mm to (190.8, 125.7), turned to -90 degrees
- moved U3 244.7 mm to (197.6, 106.0)
- moved R7 233.8 mm to (191.5, 106.8), turned to 180 degrees
- moved C8 217.3 mm to (190.7, 104.0), turned to -90 degrees
- moved C5 68.5 mm to (150.8, 224.0), turned to -90 degrees
- moved R3 51.1 mm to (151.0, 231.8), turned to 180 degrees
- moved C4 47.6 mm to (158.0, 226.5), turned to -90 degrees
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
Commit message: placement done, ESP32 footprint added
Parts:
- removed C10, C7: 2u2 100V, Capacitor_SMD:CP_Elec_6.3x5.4
- removed C14, C8: 1u 16V, Capacitor_SMD:C_0805_2012Metric_Pad1.18x1.45mm_HandSolder
- removed D2, D3: SS310, Diode_SMD:D_SMA_Handsoldering
- removed J4, J5: Molex 26013114, Connector_Molex:Molex_Mini-Fit_Jr_5569-02A2_2x01_P4.20mm_Horizontal
- removed L3, L5: 33u 2A, Inductor_SMD:L_12x12mm_H6mm
- removed R13, R7: 3k3, Resistor_SMD:R_0603_1608Metric_Pad0.98x0.95mm_HandSolder
- removed R14, R8: 20k, Resistor_SMD:R_0603_1608Metric_Pad0.98x0.95mm_HandSolder
- removed U3, U5: LM3414, PersonalDiscretes:TI_SO-PowerPAD-8_HandSolder
- added C1: 2u2 100V, Capacitor_SMD:CP_Elec_6.3x5.4, F.Cu at (183.7, 105.5)
- added C1: 2u2 100V, Capacitor_SMD:CP_Elec_6.3x5.4, F.Cu at (183.7, 119.5)
- added C1: 2u2 100V, Capacitor_SMD:CP_Elec_6.3x5.4, F.Cu at (183.7, 91.5)
- added C2: 1u 16V, Capacitor_SMD:C_0805_2012Metric_Pad1.18x1.45mm_HandSolder, F.Cu at (176.7, 96.5)
- added C2: 1u 16V, Capacitor_SMD:C_0805_2012Metric_Pad1.18x1.45mm_HandSolder, F.Cu at (176.7, 110.5)
- added C2: 1u 16V, Capacitor_SMD:C_0805_2012Metric_Pad1.18x1.45mm_HandSolder, F.Cu at (176.7, 124.5)
- added C3: 10nF 50V, Capacitor_SMD:C_0805_2012Metric_Pad1.18x1.45mm_HandSolder, F.Cu at (163.0, 111.5)
- added C4: 4u7 100V, Capacitor_SMD:C_1210_3225Metric, F.Cu at (166.8, 107.8)
- added C5: 10u 25V, Capacitor_SMD:C_0805_2012Metric_Pad1.18x1.45mm_HandSolder, F.Cu at (164.2, 115.0)
- added D1: SS310, Diode_SMD:D_SMA_Handsoldering, F.Cu at (190.4, 109.5)
- added D1: SS310, Diode_SMD:D_SMA_Handsoldering, F.Cu at (190.4, 123.5)
- added D1: SS310, Diode_SMD:D_SMA_Handsoldering, F.Cu at (190.4, 95.5)
- added J3: Molex 26013114, Connector_Molex:Molex_Mini-Fit_Jr_5569-02A2_2x01_P4.20mm_Horizontal, F.Cu at (215.8, 110.0)
- added J3: Molex 26013114, Connector_Molex:Molex_Mini-Fit_Jr_5569-02A2_2x01_P4.20mm_Horizontal, F.Cu at (215.8, 96.0)
- added J3: Molex 26013114, Connector_Molex:Molex_Mini-Fit_Jr_5569-02A2_2x01_P4.20mm_Horizontal, F.Cu at (215.8, 124.0)
- added L1: 33u 2A, Inductor_SMD:L_12x12mm_H6mm, F.Cu at (199.2, 95.8)
- added L1: 33u 2A, Inductor_SMD:L_12x12mm_H6mm, F.Cu at (199.2, 109.8)
- added L1: 33u 2A, Inductor_SMD:L_12x12mm_H6mm, F.Cu at (199.2, 123.8)
- added L2: 20uH >1.2A, Inductor_SMD:L_Taiyo-Yuden_NR-80xx, F.Cu at (157.5, 113.8)
- added R1: 3k3, Resistor_SMD:R_0603_1608Metric_Pad0.98x0.95mm_HandSolder, F.Cu at (177.4, 113.2)
- added R1: 3k3, Resistor_SMD:R_0603_1608Metric_Pad0.98x0.95mm_HandSolder, F.Cu at (177.4, 99.2)
- added R1: 3k3, Resistor_SMD:R_0603_1608Metric_Pad0.98x0.95mm_HandSolder, F.Cu at (177.4, 127.2)
- added R2: 20k, Resistor_SMD:R_0603_1608Metric_Pad0.98x0.95mm_HandSolder, F.Cu at (189.4, 115.0)
- added R2: 20k, Resistor_SMD:R_0603_1608Metric_Pad0.98x0.95mm_HandSolder, F.Cu at (189.4, 129.0)
- added R2: 20k, Resistor_SMD:R_0603_1608Metric_Pad0.98x0.95mm_HandSolder, F.Cu at (189.4, 101.0)
- added R3: 100k, Resistor_SMD:R_0603_1608Metric_Pad0.98x0.95mm_HandSolder, F.Cu at (172.0, 114.8)
- added R4: 4k7, Resistor_SMD:R_0603_1608Metric_Pad0.98x0.95mm_HandSolder, F.Cu at (171.8, 111.4)
- added R5: 100k, Resistor_SMD:R_0603_1608Metric_Pad0.98x0.95mm_HandSolder, F.Cu at (169.8, 114.8)
- added R6: 560R, Resistor_SMD:R_0603_1608Metric_Pad0.98x0.95mm_HandSolder, F.Cu at (174.0, 112.0)
- added U1: LM3414, PersonalDiscretes:TI_SO-PowerPAD-8_HandSolder, F.Cu at (183.5, 126.5)
- added U1: LM3414, PersonalDiscretes:TI_SO-PowerPAD-8_HandSolder, F.Cu at (183.5, 98.5)
- added U1: LM3414, PersonalDiscretes:TI_SO-PowerPAD-8_HandSolder, F.Cu at (183.5, 112.5)
- added U2: SY8303, Package_TO_SOT_SMD:TSOT-23-8, F.Cu at (166.5, 111.5)
- U9: footprint Package_DFN_QFN:QFN-48-1EP_7x7mm_P0.5mm_EP5.3x5.3mm -> PersonalDiscretes:ESP32-PICO-MINI-02
- moved C28 760.9 mm to (220.2, 132.5), turned to 180 degrees
- moved C27 750.1 mm to (220.2, 134.8), turned to 180 degrees
- moved R28 715.7 mm to (216.2, 139.5), turned to -90 degrees
- moved Q3 712.0 mm to (219.9, 139.5)
- moved R27 702.9 mm to (218.9, 136.8), turned to 180 degrees
- moved J1 702.7 mm to (226.3, 138.1), turned to 90 degrees
- moved R25 698.0 mm to (179.2, 145.8), turned to -90 degrees
- moved Q2 694.6 mm to (182.2, 145.8)
- moved R26 667.6 mm to (215.0, 134.5)
- moved R24 665.7 mm to (179.2, 142.2), turned to 90 degrees
- moved Q1 662.1 mm to (182.2, 142.2)
- moved Q4 654.2 mm to (214.5, 131.4), turned to 90 degrees
- moved R30 642.6 mm to (212.5, 135.2), turned to 90 degrees
- moved R29 632.8 mm to (215.0, 136.2)
- moved C25 614.3 mm to (205.5, 132.8), turned to -90 degrees
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